File: ESP12DualStepperPCB/RulleGardin.kicad_pcb (KiCad board)
At the start: 2 copper layers, 56 x 33 mm, 22 parts, among them J1 Power, J2 Conn_02x03_Odd_Even, J3 Conn_01x05, U1 ESP-12E, U2 TSR_1-2433, U3 ULN2003A

Commit message: PCB update
Parts:
- removed R10, R5, R6, R7, R8, R9: NM, Resistor_SMD:R_0805_2012Metric
- added JP1: jumper, Jumper:SolderJumper-3_P1.3mm_Open_RoundedPad1.0x1.5mm, F.Cu at (199.7, 87.4)
- added JP2: Jumper, Jumper:SolderJumper-3_P1.3mm_Open_RoundedPad1.0x1.5mm, F.Cu at (194.3, 87.4)
- added JP3: Jumper, Jumper:SolderJumper-3_P1.3mm_Open_RoundedPad1.0x1.5mm, F.Cu at (194.3, 91.2)
- added U4: AZ1117-3.3, Package_TO_SOT_SMD:SOT-223-3_TabPin2, B.Cu at (156.8, 103.4)
- moved J2 2.46 mm to (185.9, 89.7), turned to 90 degrees
Connections:
- net +3V3 renamed +3.3V
- net /EN renamed /Esp8266/EN
- net /RX renamed /Esp8266/RX
- net /TX renamed /Esp8266/TX
- net Net-(R2-Pad1) renamed /Esp8266/GPIO15
- A1 pad 2: (no net) -> unconnected-(A1-~{FLT}-Pad2)
- U1 pad 10: (no net) -> unconnected-(U1-MISO-Pad10)
- U1 pad 11: (no net) -> unconnected-(U1-GPIO9-Pad11)
- U1 pad 12: (no net) -> unconnected-(U1-GPIO10-Pad12)
- U1 pad 13: (no net) -> unconnected-(U1-MOSI-Pad13)
- U1 pad 14: (no net) -> unconnected-(U1-SCLK-Pad14)
- U1 pad 2: (no net) -> /Esp8266/AnalogIn
- U1 pad 4: (no net) -> /Esp8266/GPIO16
- U1 pad 5: (no net) -> /Esp8266/GPIO14
- U1 pad 6: (no net) -> /Esp8266/GPIO12
- U1 pad 7: (no net) -> /Esp8266/GPIO13
- U1 pad 9: (no net) -> unconnected-(U1-CS0-Pad9)
- U3 pad 10: (no net) -> unconnected-(U3-O7-Pad10)
- U3 pad 11: (no net) -> unconnected-(U3-O6-Pad11)
- U3 pad 12: (no net) -> unconnected-(U3-O5-Pad12)
Routing:
- net +3.3V: track 93.6 -> 121.6 mm
- net GNDD: track 0.00 -> 8.54 mm
- net +5V: track 117.3 -> 111.1 mm, vias 1 -> 0
- net /D0: track 40.9 -> 46.2 mm
- net Net-(A1-M2): track 21.2 -> 26.0 mm
- net /Esp8266/RX: track 9.95 -> 13.6 mm
- net /Esp8266/TX: track 9.62 -> 11.2 mm
- net /Esp8266/EN: track 33.3 -> 31.8 mm
- net Net-(A1-M1): track 19.5 -> 20.9 mm
- net /Coil2: track 9.03 -> 8.16 mm
Other:
- net class Default removed
